File: v6/dev_artix/fpga_bank1.kicad_sch (KiCad schematic)
At the start: 64 parts, among them J301 SMA-FEMALE-H, J302 SMA-FEMALE-H, J303 SMA-FEMALE-H, J304 SMA-FEMALE-H, J305 PMOD, J306 PMOD, J307 PMOD, U301 XC7A100T-CSG324, U302 S25FL256S

Commit message: Adapt numbers for easier ordering and assembling
Parts:
- C301, C302, C303, C304, C308, C309, C310, C311, C315, C316, C317, C318, C322, C323, C324, C325: value 0.47u -> 470n
- C305, C306, C312, C313, C319, C320, C326, C327: value 4.7u -> 10µ
- C307, C314, C321, C328: value 100u -> 100µ
- R305: value 49.9R -> 100R
- R306, R307, R308: value 1.5kR -> 1k5
- R313, R314, R315: value 10kR -> 10k
Changed lines of the file:
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@@
 			)
 		)
-		(property "Value" "10kR"
+		(property "Value" "10k"
 			(at 205.74 250.19 90)
 			(effects
@@
 			)
 		)
-		(property "Value" "100u"
+		(property "Value" "100µ"
 			(at 209.804 36.83 0)
 			(effects
@@
 			)
 		)
-		(property "Value" "1.5kR"
+		(property "Value" "1k5"
 			(at 109.22 213.3599 0)
 			(effects
@@
 			)
 		)
-		(property "Value" "0.47u"
+		(property "Value" "470n"
 			(at 236.474 36.83 0)
 			(effects
@@
 			)
 		)
-		(property "Value" "10kR"
+		(property "Value" "10k"
 			(at 205.74 229.87 90)
 			(effects
@@
 			)
 		)
-		(property "Value" "0.47u"
+		(property "Value" "470n"
 			(at 352.044 36.83 0)
 			(effects
@@
 			)
 		)
-		(property "Value" "0.47u"
+		(property "Value" "470n"
 			(at 272.034 36.83 0)
 			(effects
@@
 			)
 		)
-		(property "Value" "4.7u"
+		(property "Value" "10µ"
 			(at 283.464 36.83 0)
 			(effects
@@
 			)
 		)
-		(property "Value" "4.7u"
+		(property "Value" "10µ"
 			(at 188.214 36.83 0)
 			(effects
@@
 			)
 		)
-		(property "Value" "0.47u"
+		(property "Value" "470n"
 			(at 142.748 36.83 0)
 			(effects
@@
 			)
 		)
-		(property "Value" "1.5kR"
+		(property "Value" "1k5"
 			(at 123.19 213.3599 0)
 			(effects
@@
 			)
 		)
-		(property "Value" "0.47u"
+		(property "Value" "470n"
 			(at 247.904 36.83 0)
 			(effects
@@
 			)
 		)
-		(property "Value" "0.47u"
+		(property "Value" "470n"
 			(at 165.608 36.83 0)
 			(effects
@@
 			)
 		)
-		(property "Value" "0.47u"
+		(property "Value" "470n"
 			(at 154.178 36.83 0)
 			(effects
@@
 			)
 		)
-		(property "Value" "100u"
+		(property "Value" "100µ"
 			(at 396.494 36.83 0)
 			(effects
@@
 			)
 		)
-		(property "Value" "0.47u"
+		(property "Value" "470n"
 			(at 340.614 36.83 0)
 			(effects
@@
 			)
 		)
-		(property "Value" "0.47u"
+		(property "Value" "470n"
 			(at 52.324 36.83 0)
 			(effects
@@
 			)
 		)
-		(property "Value" "0.47u"
+		(property "Value" "470n"
 			(at 63.754 36.83 0)
 			(effects
@@
 			)
 		)
-		(property "Value" "0.47u"
+		(property "Value" "470n"
 			(at 75.184 36.83 0)
 			(effects
@@
 			)
 		)
-		(property "Value" "100u"
+		(property "Value" "100µ"
 			(at 305.054 36.83 0)
 			(effects
@@
 			)
 		)
-		(property "Value" "49.9R"
+		(property "Value" "100R"
 			(at 62.738 78.232 90)
 			(effects
@@
 			)
 		)
-		(property "Value" "0.47u"
+		(property "Value" "470n"
 			(at 40.894 36.83 0)
 			(effects
@@
 			)
 		)
-		(property "Value" "1.5kR"
+		(property "Value" "1k5"
 			(at 93.98 213.3599 0)
 			(effects
@@
 			)
 		)
-		(property "Value" "4.7u"
+		(property "Value" "10µ"
 			(at 199.644 36.83 0)
 			(effects
@@
 			)
 		)
-		(property "Value" "0.47u"
+		(property "Value" "470n"
 			(at 363.474 36.83 0)
 			(effects
@@
 			)
 		)
-		(property "Value" "0.47u"
+		(property "Value" "470n"
 			(at 329.184 36.83 0)
 			(effects
@@
 			)
 		)
-		(property "Value" "10kR"
+		(property "Value" "10k"
 			(at 205.74 270.51 90)
 			(effects
@@
 			)
 		)
-		(property "Value" "4.7u"
+		(property "Value" "10µ"
 			(at 294.894 36.83 0)
 			(effects
@@
 			)
 		)
-		(property "Value" "0.47u"
+		(property "Value" "470n"
 			(at 259.334 36.83 0)
 			(effects
@@
 			)
 		)
-		(property "Value" "0.47u"
+		(property "Value" "470n"
 			(at 177.038 36.83 0)
 			(effects
@@
 			)
 		)
-		(property "Value" "4.7u"
+		(property "Value" "10µ"
 			(at 86.614 36.83 0)
 			(effects
@@
 			)
 		)
-		(property "Value" "4.7u"
+		(property "Value" "10µ"
 			(at 98.044 36.83 0)
 			(effects
@@
 			)
 		)
-		(property "Value" "4.7u"
+		(property "Value" "10µ"
 			(at 386.334 36.83 0)
 			(effects
@@
 			)
 		)
-		(property "Value" "100u"
+		(property "Value" "100µ"
 			(at 108.204 36.83 0)
 			(effects
@@
 			)
 		)
-		(property "Value" "4.7u"
+		(property "Value" "10µ"
 			(at 374.904 36.83 0)
 			(effects
