File: v6/mini/mini.kicad_pcb (KiCad board)
At the start: 4 copper layers, 51 x 23 mm, 73 parts, among them J1 USB-C Receptable (16P), J2 SMA-FEMALE-H, J3 Pico Debugger (SWD), J4 SMA-FEMALE-H, U1 PAC1954T-E4Mx, U2 ADP7142AUJZ, U3 ADP7142AUJZ, U4 PMOD, U5 ICE40UP5K-SG48ITR50, U6 W25Q16JVUXIQ, U7 W25Q16JVUXIQ, U8 RP2350A, Y1 KX7_12M

Commit message: Add comments for GateMAte board
Parts:
- R1, R2, R3: value 0R82 -> 1R
- R9: value 0R1 -> 1R
