File: v6/mini/mini.kicad_pcb (KiCad board)
At the start: 4 copper layers, 51 x 23 mm, 73 parts, among them J1 USB-C Receptable (16P), J2 SMA-FEMALE-H, J3 Pico Debugger (SWD), J4 SMA-FEMALE-H, U1 PAC1954T-E4Mx, U2 ADP7142AUJZ, U3 ADP7142AUJZ, U4 PMOD, U5 ICE40UP5K-SG48ITR50, U6 W25Q16JVUXIQ, U7 W25Q16JVUXIQ, U8 RP2350A, Y1 KX7_12M

Commit message: Redesign of ENV6.mini
Parts:
- removed R12, R13: 10k, Resistor_SMD:R_0402_1005Metric
- removed R14: 5k1, Resistor_SMD:R_0402_1005Metric
- removed U3: ADP7142AUJZ, Package_TO_SOT_SMD:TSOT-23-5
- added U9: TLV73333PDBV, Package_TO_SOT_SMD:SOT-23-5, B.Cu at (132.5, 99.6)
- C12: value 100n -> 10u
- C2, C3, C4, C5: footprint Capacitor_SMD:C_0805_2012Metric -> Capacitor_SMD:C_0402_1005Metric
- R1, R2, R3: footprint Resistor_SMD:R_0402_1005Metric -> Resistor_SMD:R_0603_1608Metric
- R11, R17, R18, R19, R20, R21, R22: value 10k -> 5k1
- R9: value 1R -> 750R
- U1: footprint custom_library:QFN-16-1EP_4x4mm_P0.65mm_EP2.1x2.1mm -> sensors:VQFN-16-1EP_3x3mm_P0.5mm_EP1.1x1.1mm
- U2: value ADP7142AUJZ -> TLV73312PDBV; footprint Package_TO_SOT_SMD:TSOT-23-5 -> Package_TO_SOT_SMD:SOT-23-5
- moved C5 14.2 mm to (145.3, 102.9), turned to 90 degrees
- moved C2 11.8 mm to (133.5, 102.9), turned to 90 degrees
- moved C3 6.42 mm to (133.0, 97.0), turned to 0 degrees
- moved C1 0.70 mm to (141.0, 96.3), turned to -90 degrees
- moved C4 0.67 mm to (144.8, 97.0), turned to 0 degrees
- moved C12 0.64 mm to (146.7, 93.7), turned to 0 degrees
- moved C13 0.59 mm to (136.8, 97.5)
- moved R2 0.57 mm to (135.8, 96.9)
- moved R1 0.48 mm to (147.5, 96.8)
- moved R3 0.38 mm to (130.7, 102.4)
- moved R16 0.07 mm to (153.7, 88.6)
- moved U2 0.06 mm to (144.3, 99.6)
- moved D1 0.06 mm to (156.1, 88.4)
Connections:
- C2 pad 1: VPWR_USB -> GNDD
- C2 pad 2: GNDD -> VPWR_USB
- C3 pad 1: VPWR_USB -> GNDD
- C3 pad 2: GNDD -> /Connectors/VLDO_3V3
- C4 pad 1: /Connectors/VLDO_1V2 -> GNDD
- C4 pad 2: GNDD -> /Connectors/VLDO_1V2
- C5 pad 1: /Connectors/VLDO_3V3 -> GNDD
- C5 pad 2: GNDD -> VPWR_USB
- U2 pad 4: /Connectors/VLDO_1V2 -> unconnected-(U2-NC-Pad4)
Routing:
- net Net-(U3-SENSE/ADJ): track 5.05 -> 0.00 mm
- net /Connectors/VLDO_1V2: track 14.0 -> 10.4 mm
- net VDD: track 50.8 -> 48.9 mm, vias 30 -> 29
- net /Connectors/VLDO_3V3: track 11.8 -> 10.5 mm
- net Net-(R12-Pad1): track 1.00 -> 0.00 mm
- net Net-(U1-SLOW): track 1.77 -> 1.04 mm
- net VPWR_USB: track 27.4 -> 28.1 mm
- net +1V2: track 14.5 -> 15.1 mm
- net Net-(U1-ADDRSEL): track 0.30 -> 0.85 mm
- net GNDD: track 1.30 -> 1.82 mm, vias 200 -> 212
- net /Connectors/USB_PWRIN: track 30.7 -> 31.2 mm
Other:
- board text added: "elasticAI.hardware ENV6 mini 1v1 (c) 2026"
- board text removed: "elasticAI.hardware ENV6 mini 1v0 (c) 2026"

Commit message: Add fourth PAC sensor to ENV6mini
Parts:
- added R12: 1R, Resistor_SMD:R_0603_1608Metric, F.Cu at (149.7, 103.8)
- moved C6 1.17 mm to (151.8, 103.2), turned to 90 degrees
Connections:
- C6 pad 1: VDD -> VCCQ
- U1 pad 11: unconnected-(U1-SENSE1+-Pad11) -> VDD
- U1 pad 12: unconnected-(U1-SENSE1--Pad12) -> VCCQ
- U4 pad 1: VDD -> VCCQ
- U4 pad 2: VDD -> VCCQ
Routing:
- net VCCQ: track 0.00 -> 16.9 mm
- net VDD: track 48.9 -> 56.5 mm
- net GNDD: vias 212 -> 210

Commit message: Fixed errors in ENV6mini
Parts:
- removed R11: 5k1, Resistor_SMD:R_0402_1005Metric
- added R27: 5k1, Resistor_SMD:R_0402_1005Metric, F.Cu at (144.8, 98.0)
- added R28: 5k1, Resistor_SMD:R_0402_1005Metric, F.Cu at (143.8, 98.0)
- added REF**: Fiducial_0.75mm_Mask1.5mm, maker:Fiducial_0.75mm_Mask1.5mm, F.Cu at (117.5, 103.2)
- added REF**: Fiducial_0.75mm_Mask1.5mm, maker:Fiducial_0.75mm_Mask1.5mm, F.Cu at (164.8, 84.0)
- added REF**: Fiducial_0.75mm_Mask1.5mm, maker:Fiducial_0.75mm_Mask1.5mm, F.Cu at (164.8, 103.2)
- added REF**: Fiducial_0.75mm_Mask1.5mm, maker:Fiducial_0.75mm_Mask1.5mm, B.Cu at (164.8, 84.0)
- added REF**: Fiducial_0.75mm_Mask1.5mm, maker:Fiducial_0.75mm_Mask1.5mm, B.Cu at (164.8, 103.2)
- added REF**: Fiducial_0.75mm_Mask1.5mm, maker:Fiducial_0.75mm_Mask1.5mm, B.Cu at (117.3, 84.0)
- R10: moved to F.Cu
- moved R24 2.44 mm to (132.5, 87.6)
- moved R10 1.91 mm to (142.0, 96.3), turned to 90 degrees
- moved G*** 1.78 mm to (161.2, 102.2)
- moved C15 1.32 mm to (130.6, 87.6)
- moved J2 1.21 mm to (158.8, 84.1)
- moved R15 0.74 mm to (158.9, 87.9), turned to 90 degrees
Connections:
- U1 pad 16: Net-(U1-~{PWRDN}) -> EN_PAC
- U5 pad 25: unconnected-(U5-IOT_36B-Pad25) -> I2C_FPGA_SCL
- U5 pad 26: unconnected-(U5-IOT_39A-Pad26) -> I2C_FPGA_SDA
- U5 pad 28: unconnected-(U5-IOT_41A-Pad28) -> FPGA_GPIO2
- U5 pad 35: I2C_SCL -> unconnected-(U5-IOT_46B_G0-Pad35)
- U5 pad 36: I2C_SDA -> unconnected-(U5-IOT_48B-Pad36)
- U8 pad 12: unconnected-(U8-GPIO_08-Pad12) -> EN_PAC
- U8 pad 2: unconnected-(U8-GPIO_00-Pad2) -> I2C_FPGA_SDA
- U8 pad 3: unconnected-(U8-GPIO_01-Pad3) -> I2C_FPGA_SCL
- U8 pad 8: unconnected-(U8-GPIO_05-Pad8) -> FPGA_GPIO2
Routing:
- net I2C_FPGA_SDA: track 0.00 -> 19.2 mm, vias 0 -> 2
- net I2C_FPGA_SCL: track 0.00 -> 17.7 mm, vias 0 -> 2
- net I2C_SDA: track 19.0 -> 4.30 mm, vias 2 -> 1
- net FPGA_GPIO2: track 0.00 -> 14.5 mm, vias 0 -> 2
- net I2C_SCL: track 17.2 -> 4.08 mm, vias 2 -> 1
- net EN_PAC: track 0.00 -> 10.6 mm, vias 0 -> 2
- net Net-(U8-GPIO_29_ADC3): track 4.20 -> 1.13 mm
- net Net-(U1-~{PWRDN}): track 2.80 -> 0.00 mm
- net Net-(J4-SIG): track 2.71 -> 4.25 mm
- net Net-(U1-SLOW): track 1.04 -> 2.15 mm, vias 1 -> 0
- net Net-(U5-IOB_5B): track 9.91 -> 8.84 mm
- net Net-(J2-SIG): track 3.81 -> 2.77 mm
- net GNDD: track 1.82 -> 2.69 mm, vias 210 -> 197
- net PWR_EN_FPGA: track 11.1 -> 10.4 mm
- net VDD: track 56.5 -> 56.1 mm, vias 29 -> 30
