File: v6/mini/connector.kicad_sch (KiCad schematic)
At the start: 25 parts, among them J1 USB-C Receptable (16P), U1 PAC1954T-E4Mx, U2 ADP7142AUJZ, U3 ADP7142AUJZ

Commit message: Redesign of ENV6.mini
Parts:
- removed C2, C3, C4, C5: 10u, Capacitor_SMD:C_0805_2012Metric, symbol passive:C0805
- removed R12, R13: 10k, Resistor_SMD:R_0402_1005Metric, symbol passive:R0402
- removed R14: 5k1, Resistor_SMD:R_0402_1005Metric, symbol passive:R0402
- removed U2, U3: ADP7142AUJZ, Package_TO_SOT_SMD:TSOT-23-5, symbol Regulator_Linear:ADP7142AUJZ
- added C2, C3, C4, C5: 10u, Capacitor_SMD:C_0402_1005Metric, symbol passive:C0402
- added U2: TLV73312PDBV, Package_TO_SOT_SMD:SOT-23-5, symbol Regulator_Linear:TLV73312PDBV
- added U9: TLV73333PDBV, Package_TO_SOT_SMD:SOT-23-5, symbol Regulator_Linear:TLV73333PDBV
- R1, R2, R3: footprint Resistor_SMD:R_0402_1005Metric -> Resistor_SMD:R_0603_1608Metric
- R11: value 10k -> 5k1
- R9: value 1R -> 750R
- U1: footprint custom_library:QFN-16-1EP_4x4mm_P0.65mm_EP2.1x2.1mm -> sensors:VQFN-16-1EP_3x3mm_P0.5mm_EP1.1x1.1mm
Connections:
- net GNDD: now also C2.1, C3.1, C4.1, C5.1, U2.2 (GND), U9.2 (GND)
- net PWR_EN_FPGA: now also U2.3 (EN)
- net VLDO_1V2: now also C4.2, U2.5 (OUT)
- net VLDO_3V3: now also C3.2, U9.5 (OUT)
- net VPWR_USB: now also C2.2, C5.2, U2.1 (IN), U9.1 (IN), U9.3 (EN)
Other:
- note added: "(0.1% accuracy, 1W, max 1A)"
- note removed: "find a link to buy sense resistors (0.1% accuracy, high power budget)"
- company: (none) -> UDE-IES
- title: (none) -> elasticAI.hardware (ENV6.mini)

Commit message: Add fourth PAC sensor to ENV6mini
Parts:
- added R12: 1R, Resistor_SMD:R_0603_1608Metric, symbol passive:R0402
Connections:
- net VDD: now also U1.11 (SENSE1+), R12.2
- net VCCQ: now reaches U1.12 (SENSE1-)
- net VCCQ: now also R12.1
- no-connect marks 5 -> 3

Commit message: Fixed errors in ENV6mini
Parts:
- removed R11: 5k1, Resistor_SMD:R_0402_1005Metric, symbol passive:R0402
Connections:
- net EN_PAC: now reaches U1.16 (~{PWRDN})
Changed lines of the file:
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@@
-	)
-	(junction
-		(at 114.3 132.08)
-		(diameter 0)
-		(color 0 0 0 0)
 	)
 	(junction
@@
 	(wire
 		(pts
-			(xy 114.3 143.51) (xy 114.3 146.05)
-		)
-		(stroke
-			(width 0)
-			(type default)
-		)
-	)
-	(wire
-		(pts
 			(xy 217.17 137.16) (xy 217.17 140.97)
 		)
@@
 	(wire
 		(pts
-			(xy 92.71 146.05) (xy 114.3 146.05)
-		)
-		(stroke
-			(width 0)
-			(type default)
-		)
-	)
-	(wire
-		(pts
 			(xy 110.49 163.83) (xy 110.49 166.37)
 		)
@@
 	(wire
 		(pts
+			(xy 92.71 146.05) (xy 93.98 146.05)
+		)
+		(stroke
+			(width 0)
+			(type default)
+		)
+	)
+	(wire
+		(pts
 			(xy 44.45 152.4) (xy 67.31 152.4)
 		)
@@
 	(wire
 		(pts
-			(xy 114.3 132.08) (xy 114.3 135.89)
-		)
-		(stroke
-			(width 0)
-			(type default)
-		)
-	)
-	(wire
-		(pts
 			(xy 41.91 142.24) (xy 41.91 143.51)
 		)
@@
 	(wire
 		(pts
-			(xy 92.71 132.08) (xy 114.3 132.08)
+			(xy 92.71 132.08) (xy 125.73 132.08)
 		)
 		(stroke
@@
 		(pts
 			(xy 95.25 162.56) (xy 95.25 165.1)
-		)
-		(stroke
-			(width 0)
-			(type default)
-		)
-	)
-	(wire
-		(pts
-			(xy 114.3 132.08) (xy 125.73 132.08)
 		)
 		(stroke
@@
 		(property "Intersheetrefs" "${INTERSHEET_REFS}"
 			(at 92.8528 73.66 0)
+			(hide yes)
+			(show_name no)
+			(do_not_autoplace no)
+			(effects
+				(font
+					(size 1.27 1.27)
+				)
+				(justify left)
+			)
+		)
+	)
+	(global_label "EN_PAC"
+		(shape input)
+		(at 93.98 146.05 0)
+		(fields_autoplaced yes)
+		(effects
+			(font
+				(size 1.27 1.27)
+			)
+			(justify left)
+		)
+		(property "Intersheetrefs" "${INTERSHEET_REFS}"
+			(at 104.0409 146.05 0)
 			(hide yes)
 			(show_name no)
@@
 					(unit 1)
 				)
-			)
-		)
-	)
-	(symbol
-		(lib_id "passive:R0402")
-		(at 114.3 139.7 0)
-		(unit 1)
-		(body_style 1)
-		(exclude_from_sim no)
-		(in_bom yes)
-		(on_board yes)
-		(in_pos_files yes)
-		(dnp no)
-		(fields_autoplaced yes)
-		(property "Reference" "R11"
-			(at 116.84 138.4299 0)
-			(show_name no)
-			(do_not_autoplace no)
-			(effects
-				(font
-					(size 1.27 1.27)
-				)
-				(justify left)
-			)
-		)
-		(property "Value" "5k1"
-			(at 116.84 140.9699 0)
-			(show_name no)
-			(do_not_autoplace no)
-			(effects
-				(font
-					(size 1.27 1.27)
-				)
-				(justify left)
-			)
-		)
-		(property "Footprint" "Resistor_SMD:R_0402_1005Metric"
-			(at 112.522 139.7 90)
-			(hide yes)
-			(show_name no)
-			(do_not_autoplace no)
-			(effects
-				(font
-					(size 1.27 1.27)
-				)
-			)
-		)
-		(property "Datasheet" ""
-			(at 114.3 139.7 0)
-			(hide yes)
-			(show_name no)
-			(do_not_autoplace no)
-			(effects
-				(font
-					(size 1.27 1.27)
-				)
-			)
-		)
-		(property "Description" "Resistor"
-			(at 114.3 139.7 0)
-			(hide yes)
-			(show_name no)
-			(do_not_autoplace no)
-			(effects
-				(font
-					(size 1.27 1.27)
-				)
-			)
-		)
-		(pin "2"
-		)
-		(pin "1"
-		)
-		(instances
-			(project "mini"
-				(path "/cad3e569-714f-4d3a-be70-27b5cd29ede2/cfce4952-8973-4417-93ad-c631a1c587c4"
-					(reference "R11")
-					(unit 1)
-				)
