File: v6/mini/fpga.kicad_sch (KiCad schematic)
At the start: 19 parts, among them J2 SMA-FEMALE-H, U4 PMOD, U5 ICE40UP5K-SG48ITR50, U6 W25Q16JVUXIQ

Commit message: Redesign of ENV6.mini
Parts:
- C12: value 100n -> 10u
- R17, R18, R19, R20, R21: value 10k -> 5k1
Other:
- company: (none) -> UDE-IES
- title: (none) -> elasticAI.hardware (ENV6.mini)
Changed lines of the file:
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@@
 	(generator_version "10.0")
 	(paper "A4")
+	(title_block
+		(title "elasticAI.hardware (ENV6.mini)")
+		(date "2026-07-03")
+		(rev "1v1")
+		(company "UDE-IES")
+	)
 	(text "SPI_MISO"
 		(exclude_from_sim no)
@@
 			)
 		)
-		(property "Value" "10k"
+		(property "Value" "5k1"
 			(at 248.92 67.3099 0)
 			(show_name no)
@@
 			)
 		)
-		(property "Value" "10k"
+		(property "Value" "5k1"
 			(at 209.55 72.3899 0)
 			(show_name no)
@@
 			)
 		)
-		(property "Value" "10k"
+		(property "Value" "5k1"
 			(at 266.7 67.3099 0)
 			(show_name no)
@@
 	)
 	(symbol
-		(lib_id "passive:C0402")
-		(at 194.31 119.38 0)
-		(unit 1)
-		(body_style 1)
-		(exclude_from_sim no)
-		(in_bom yes)
-		(on_board yes)
-		(in_pos_files yes)
-		(dnp no)
-		(fields_autoplaced yes)
-		(property "Reference" "C12"
-			(at 198.12 118.1099 0)
-			(show_name no)
-			(do_not_autoplace no)
-			(effects
-				(font
-					(size 1.27 1.27)
-				)
-				(justify left)
-			)
-		)
-		(property "Value" "100n"
-			(at 198.12 120.6499 0)
-			(show_name no)
-			(do_not_autoplace no)
-			(effects
-				(font
-					(size 1.27 1.27)
-				)
-				(justify left)
-			)
-		)
-		(property "Footprint" "Capacitor_SMD:C_0402_1005Metric"
-			(at 195.2752 123.19 0)
-			(hide yes)
-			(show_name no)
-			(do_not_autoplace no)
-			(effects
-				(font
-					(size 1.27 1.27)
-				)
-			)
-		)
-		(property "Datasheet" ""
-			(at 194.31 119.38 0)
-			(hide yes)
-			(show_name no)
-			(do_not_autoplace no)
-			(effects
-				(font
-					(size 1.27 1.27)
-				)
-			)
-		)
-		(property "Description" "Unpolarized capacitor"
-			(at 194.31 119.38 0)
-			(hide yes)
-			(show_name no)
-			(do_not_autoplace no)
-			(effects
-				(font
-					(size 1.27 1.27)
-				)
-			)
-		)
-		(pin "1"
-		)
-		(pin "2"
-		)
-		(instances
-			(project "mini"
-				(path "/cad3e569-714f-4d3a-be70-27b5cd29ede2/7b1405f2-b11d-4a7e-9ddf-9f97b84483e2"
-					(reference "C12")
-					(unit 1)
-				)
-			)
-			(project "stim_platform"
-				(path "/f29f7d6f-2c6e-471f-bb52-1b8a168ace2f/4ff046b9-f5cc-46e0-9aab-5f3ebcdb09bf"
-					(reference "C36")
-					(unit 1)
-				)
-			)
-		)
-	)
-	(symbol
 		(lib_id "passive:R0402")
 		(at 255.27 66.04 0)
@@
 			)
 		)
-		(property "Value" "10k"
+		(property "Value" "5k1"
 			(at 257.81 67.3099 0)
 			(show_name no)
@@
 	)
 	(symbol
+		(lib_id "passive:C0402")
+		(at 194.31 119.38 0)
+		(unit 1)
+		(body_style 1)
+		(exclude_from_sim no)
+		(in_bom yes)
+		(on_board yes)
+		(in_pos_files yes)
+		(dnp no)
+		(fields_autoplaced yes)
+		(property "Reference" "C12"
+			(at 198.12 118.1099 0)
+			(show_name no)
+			(do_not_autoplace no)
+			(effects
+				(font
+					(size 1.27 1.27)
+				)
+				(justify left)
+			)
+		)
+		(property "Value" "10u"
+			(at 198.12 120.6499 0)
+			(show_name no)
+			(do_not_autoplace no)
+			(effects
+				(font
+					(size 1.27 1.27)
+				)
+				(justify left)
+			)
+		)
+		(property "Footprint" "Capacitor_SMD:C_0402_1005Metric"
+			(at 195.2752 123.19 0)
+			(hide yes)
+			(show_name no)
+			(do_not_autoplace no)
+			(effects
+				(font
+					(size 1.27 1.27)
+				)
+			)
+		)
+		(property "Datasheet" ""
+			(at 194.31 119.38 0)
+			(hide yes)
+			(show_name no)
+			(do_not_autoplace no)
+			(effects
+				(font
+					(size 1.27 1.27)
+				)
+			)
+		)
+		(property "Description" "Unpolarized capacitor"
+			(at 194.31 119.38 0)
+			(hide yes)
+			(show_name no)
+			(do_not_autoplace no)
+			(effects
+				(font
+					(size 1.27 1.27)
+				)
+			)
+		)
+		(pin "1"
+		)
+		(pin "2"
+		)
+		(instances
+			(project "mini"
+				(path "/cad3e569-714f-4d3a-be70-27b5cd29ede2/7b1405f2-b11d-4a7e-9ddf-9f97b84483e2"
+					(reference "C12")
+					(unit 1)
+				)
+			)
+		)
+	)
+	(symbol
 		(lib_id "fpga:ICE40UP5K-SG48ITR50")
 		(at 107.95 102.87 0)
@@
 			)
 		)
-		(property "Value" "10k"
+		(property "Value" "5k1"
 			(at 200.66 72.3899 0)
 			(show_name no)

Commit message: Add fourth PAC sensor to ENV6mini
Connections:
- net VDD: no longer C6.1, U4.1 (VCC), U4.2 (VCC)
- new net VCCQ: C6.1, U4.1 (VCC), U4.2 (VCC)
Changed lines of the file:
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@@
-	(symbol
-		(lib_id "power:VDD")
-		(at 26.67 54.61 0)
-		(mirror y)
-		(unit 1)
-		(body_style 1)
-		(exclude_from_sim no)
-		(in_bom yes)
-		(on_board yes)
-		(in_pos_files yes)
-		(dnp no)
-		(fields_autoplaced yes)
-		(property "Reference" "#PWR014"
-			(at 26.67 58.42 0)
-			(hide yes)
-			(show_name no)
-			(do_not_autoplace no)
-			(effects
-				(font
-					(size 1.27 1.27)
-				)
-			)
-		)
-		(property "Value" "VDD"
-			(at 26.67 49.53 0)
-			(show_name no)
-			(do_not_autoplace no)
-			(effects
-				(font
-					(size 1.27 1.27)
-				)
-			)
-		)
-		(property "Footprint" ""
-			(at 26.67 54.61 0)
-			(hide yes)
-			(show_name no)
-			(do_not_autoplace no)
-			(effects
-				(font
-					(size 1.27 1.27)
-				)
-			)
-		)
-		(property "Datasheet" ""
-			(at 26.67 54.61 0)
-			(hide yes)
-			(show_name no)
-			(do_not_autoplace no)
-			(effects
-				(font
-					(size 1.27 1.27)
-				)
-			)
-		)
-		(property "Description" "Power symbol creates a global label with name \"VDD\""
-			(at 26.67 54.61 0)
-			(hide yes)
-			(show_name no)
-			(do_not_autoplace no)
-			(effects
-				(font
-					(size 1.27 1.27)
-				)
-			)
-		)
-		(pin "1"
-		)
-		(instances
-			(project "mini"
-				(path "/cad3e569-714f-4d3a-be70-27b5cd29ede2/7b1405f2-b11d-4a7e-9ddf-9f97b84483e2"
-					(reference "#PWR014")
-					(unit 1)
-				)
-			)
-		)
-	)
 	(symbol
 		(lib_id "power:VDD")
@@
 					(unit 1)
 				)
+			)
+		)
+	)
+	(symbol
+		(lib_id "power:VCCQ")
+		(at 26.67 54.61 0)
+		(unit 1)
+		(body_style 1)
+		(exclude_from_sim no)
+		(in_bom yes)
+		(on_board yes)
+		(in_pos_files yes)
+		(dnp no)
+		(fields_autoplaced yes)
+		(property "Reference" "#PWR014"
+			(at 26.67 58.42 0)
+			(hide yes)
+			(show_name no)
+			(do_not_autoplace no)
+			(effects
+				(font
+					(size 1.27 1.27)
+				)
+			)
+		)
+		(property "Value" "VCCQ"
+			(at 26.67 49.53 0)
+			(show_name no)
+			(do_not_autoplace no)
+			(effects
+				(font
+					(size 1.27 1.27)
+				)
+			)
+		)
+		(property "Footprint" ""
+			(at 26.67 54.61 0)
+			(hide yes)
+			(show_name no)
+			(do_not_autoplace no)
+			(effects
+				(font
+					(size 1.27 1.27)
+				)
+			)
+		)
+		(property "Datasheet" ""
+			(at 26.67 54.61 0)
+			(hide yes)
+			(show_name no)
+			(do_not_autoplace no)
+			(effects
+				(font
+					(size 1.27 1.27)
+				)
+			)
+		)
+		(property "Description" "Power symbol creates a global label with name \"VCCQ\""
+			(at 26.67 54.61 0)
+			(hide yes)
+			(show_name no)
+			(do_not_autoplace no)
+			(effects
+				(font
+					(size 1.27 1.27)
+				)
+			)
+		)
+		(pin "1"
+		)
+		(instances
+			(project "mini"
+				(path "/cad3e569-714f-4d3a-be70-27b5cd29ede2/7b1405f2-b11d-4a7e-9ddf-9f97b84483e2"
+					(reference "#PWR014")
+					(unit 1)
+				)

Commit message: Fixed errors in ENV6mini
Connections:
- net I2C_FPGA_SCL: now reaches U5.25 (IOT_36B)
- net I2C_FPGA_SDA: now reaches U5.26 (IOT_39A)
- net FPGA_GPIO2: now reaches U5.28 (IOT_41A)
- net I2C_SCL: no longer names the net of U5.35 (IOT_46B_G0)
- net I2C_SDA: no longer names the net of U5.36 (IOT_48B)
- no-connect marks 15 -> 14
Changed lines of the file:
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@@
+	)
+	(no_connect
+		(at 80.01 100.33)
 	)
 	(no_connect
@@
 	)
 	(no_connect
-		(at 80.01 87.63)
-	)
-	(no_connect
 		(at 80.01 138.43)
-	)
-	(no_connect
-		(at 80.01 85.09)
 	)
 	(no_connect
@@
 	)
 	(no_connect
+		(at 80.01 102.87)
+	)
+	(no_connect
 		(at 80.01 80.01)
 	)
@@
 		(at 80.01 135.89)
 	)
-	(no_connect
-		(at 80.01 77.47)
-	)
 	(wire
 		(pts
@@
 	(wire
 		(pts
-			(xy 67.31 100.33) (xy 80.01 100.33)
-		)
-		(stroke
-			(width 0)
-			(type default)
-		)
-	)
-	(wire
-		(pts
 			(xy 135.89 102.87) (xy 146.05 102.87)
 		)
@@
 	(wire
 		(pts
-			(xy 67.31 102.87) (xy 80.01 102.87)
-		)
-		(stroke
-			(width 0)
-			(type default)
-		)
-	)
-	(wire
-		(pts
 			(xy 68.58 118.11) (xy 80.01 118.11)
 		)
@@
 	(wire
 		(pts
+			(xy 78.74 85.09) (xy 80.01 85.09)
+		)
+		(stroke
+			(width 0)
+			(type default)
+		)
+	)
+	(wire
+		(pts
 			(xy 49.53 69.85) (xy 63.5 69.85)
 		)
@@
 	(wire
 		(pts
+			(xy 78.74 87.63) (xy 80.01 87.63)
+		)
+		(stroke
+			(width 0)
+			(type default)
+		)
+	)
+	(wire
+		(pts
 			(xy 49.53 57.15) (xy 63.5 57.15)
 		)
@@
 		(pts
 			(xy 146.05 48.26) (xy 149.86 48.26)
+		)
+		(stroke
+			(width 0)
+			(type default)
+		)
+	)
+	(wire
+		(pts
+			(xy 77.47 77.47) (xy 80.01 77.47)
 		)
 		(stroke
@@
 		)
 	)
-	(global_label "I2C_SCL"
-		(shape bidirectional)
-		(at 67.31 100.33 180)
+	(global_label "I2C_FPGA_SCL"
+		(shape output)
+		(at 77.47 77.47 180)
 		(fields_autoplaced yes)
 		(effects
@@
 		)
 		(property "Intersheetrefs" "${INTERSHEET_REFS}"
-			(at 55.654 100.33 0)
+			(at 61.2405 77.47 0)
 			(hide yes)
 			(show_name no)
@@
 		)
 	)
-	(global_label "I2C_SDA"
-		(shape bidirectional)
-		(at 67.31 102.87 180)
-		(fields_autoplaced yes)
-		(effects
-			(font
-				(size 1.27 1.27)
-			)
-			(justify right)
-		)
-		(property "Intersheetrefs" "${INTERSHEET_REFS}"
-			(at 55.5935 102.87 0)
-			(hide yes)
-			(show_name no)
-			(do_not_autoplace no)
-			(effects
-				(font
-					(size 1.27 1.27)
-				)
-				(justify right)
-			)
-		)
-	)
 	(global_label "FPGA_FLASH_SO"
 		(shape output)
@@
 		)
 	)
+	(global_label "I2C_FPGA_SDA"
+		(shape bidirectional)
+		(at 78.74 85.09 180)
+		(fields_autoplaced yes)
+		(effects
+			(font
+				(size 1.27 1.27)
+			)
+			(justify right)
+		)
+		(property "Intersheetrefs" "${INTERSHEET_REFS}"
+			(at 61.3387 85.09 0)
+			(hide yes)
+			(show_name no)
+			(do_not_autoplace no)
+			(effects
+				(font
+					(size 1.27 1.27)
+				)
+				(justify right)
+			)
+		)
+	)
 	(global_label "FPGA_FLASH_SI"
 		(shape input)
@@
 			(hide yes)
 			(show_name no)
+			(do_not_autoplace no)
+			(effects
+				(font
+					(size 1.27 1.27)
+				)
+				(justify right)
+			)
+		)
+	)
+	(global_label "FPGA_GPIO2"
+		(shape bidirectional)
+		(at 78.74 87.63 180)
+		(fields_autoplaced yes)
+		(effects
+			(font
+				(size 1.27 1.27)
+			)
+			(justify right)
+		)
+		(property "Intersheetrefs" "${INTERSHEET_REFS}"
+			(at 63.2739 87.63 0)
+			(hide yes)
+			(show_name no)
