File: v6/mini/mcu.kicad_sch (KiCad schematic)
At the start: 28 parts, among them J3 Pico Debugger (SWD), J4 SMA-FEMALE-H, U7 W25Q16JVUXIQ, U8 RP2350A, Y1 KX7_12M

Commit message: Redesign of ENV6.mini
Parts:
- R22: value 10k -> 5k1
Other:
- company: (none) -> UDE-IES
- title: (none) -> elasticAI.hardware (ENV6.mini)
Changed lines of the file:
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@@
 	(generator_version "10.0")
 	(paper "A4")
+	(title_block
+		(title "elasticAI.hardware (ENV6.mini)")
+		(date "2026-07-03")
+		(rev "1v1")
+		(company "UDE-IES")
+	)
 	(text "~{CS}"
 		(exclude_from_sim no)
@@
 			)
 		)
-		(property "Value" "10k"
+		(property "Value" "5k1"
 			(at 114.3 130.81 90)
 			(show_name no)
@@
 		(property "Reference" "S2"
 			(at 129.54 92.71 90)
-			(hide yes)
 			(show_name no)
 			(do_not_autoplace no)
@@
 	)
 	(symbol
-		(lib_name "Tactile Button_1")
 		(lib_id "connectors:Tactile Button")
 		(at 100.33 132.08 0)

Commit message: Fixed errors in ENV6mini
Parts:
- added R27, R28: 5k1, Resistor_SMD:R_0402_1005Metric, symbol passive:R0402
Connections:
- net VDD: now also R27.1, R28.1
- net EN_PAC: now reaches U8.12 (GPIO_08)
- net I2C_FPGA_SDA: now reaches U8.2 (GPIO_00)
- net I2C_FPGA_SDA: now also R27.2
- net I2C_FPGA_SCL: now reaches U8.3 (GPIO_01)
- net I2C_FPGA_SCL: now also R28.2
- net FPGA_GPIO2: now reaches U8.8 (GPIO_05)
- no-connect marks 12 -> 8
Other:
- note added: "i2c0"
- moved on the sheet: D2
