File: v6/ENV6_DemoBoard_1/Power.kicad_sch (KiCad schematic)
At the start: 42 parts, among them IC301 LP8758-A2EA-YFFR, U301 BQ25188, U302 TPSM8310x

Commit message: first rev Base Board pcb layout
Parts:
- removed C321, C322: 10u, Capacitor_SMD:C_0402_1005Metric, symbol passive:C0402
- removed IC301: LP8758-A2EA-YFFR, custom_library:BGA35C40P5X7_213X288X62, symbol power_devices:LP8758A2EAYFFR
- removed L303, L304: 0.47uH, Inductor_SMD:L_1008_2520Metric, symbol Device:L
- removed R305: 10k, Resistor_SMD:R_0402_1005Metric, symbol passive:R0402
- added IC301: LP873300RHDTQ1, custom_library:QFN50P500X500X80-29N, symbol LP873300RHDTQ1:LP873300RHDTQ1
- added NT301: NetTie_2, NetTie:NetTie-2_SMD_Pad0.5mm, symbol Device:NetTie_2
- renumbered C323 to C321, C324 to C322, R306 to R305, R307 to R306
Connections:
- net GND: now also IC301.15 (PGND_B1_1), IC301.16 (PGND_B1_2), IC301.20 (PGND_B0_1), IC301.21 (PGND_B0_2), NT301.1; no longer C312.1, C313.1, C314.1, C315.1, C316.1
- net GP0/I2C0_SDA: now also IC301.18 (SDA)
- net GP1/I2C0_SCL: now also IC301.17 (SCL)
- net PSU_OUT1: now also C317.2, C319.2, IC301.2 (FB_B0); no longer C311.2, C312.2
- net PSU_OUT2: now also C318.2, C320.2, IC301.3 (FB_B1); no longer C314.2, C315.2
- net PSU_OUT3: now also C315.2, IC301.1 (VOUT_LDO0); no longer C317.2, C318.2
- net PSU_OUT4: now also C316.2, IC301.7 (VOUT_LDO1); no longer C320.2
- net VFPGA_IN: now also C311.2, C312.2, C314.2, IC301.11 (VIN_B1_1), IC301.12 (VIN_B1_2), IC301.24 (VIN_B0_1), IC301.25 (VIN_B0_2), IC301.28 (VIN_LDO0), IC301.5 (VANA), IC301.8 (VIN_LDO1); no longer C316.2, C319.2
- net at L302.1: now also IC301.13 (SW_B1_1), IC301.14 (SW_B1_2)
- net at L301.1: now also IC301.22 (SW_B0_1), IC301.23 (SW_B0_2)
- new net AGND: C312.1, C313.1, C314.1, C315.1, C316.1, IC301.19 (SGND), IC301.29 (EP), IC301.4 (AGND), NT301.2
- no-connect marks 6 -> 8
Other:
- note added: "Appliaction Board"
- note added: "FPGA AUX"
- note added: "FPGA Bank"
- note added: "FPGA Core"
- note removed: "1.0 - 1.2 V / FPGA core"
- note removed: "1.8 V - 1.2 V / FPGA core"
- note removed: "3.3 V - 1.8 V / FPGA bank"
- note removed: "3.3V / FPGA"
- note removed: "Can we use all pins also using I2C? If yes, remove all And what happens with them if we do not use it? EN_BUCKn in Registers can Enable BUCKn without EN1/2 Reset can be software commanded from Reg 0x16 nRST Low = shutdown. nRST High = startup. Pull up nRST."
- note removed: "Can we use also the same with three channels? only 4 outputs availabe, to make it 3 needs to combine 2 outputs into 1"
