File: v6/ENV6_DemoBoard_1/ENV6_DemoBoard_1.kicad_sch (KiCad schematic)
At the start: 0 parts

Commit message: first rev Base Board pcb layout
Other:
- sheet Connector ports: added PSU1, PSU2, PSU3, PSU4; removed V1, V2, V3, V4
- sheet Peripherals ports: added PSU1, PSU2, PSU3, PSU4; removed V1, V2, V3, V4
Changed lines of the file:
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@@
 (kicad_sch
-	(version 20250114)
+	(version 20260306)
 	(generator "eeschema")
-	(generator_version "9.0")
+	(generator_version "10.0")
 	(paper "A4")
 	(rectangle
@@
 		)
 		(fill
-			(color 0 0 0 0.0000)
+			(color 0 0 0 0)
 		)
 		(property "Sheetname" "Peripherals"
 			(at 24.13 28.4984 0)
+			(show_name no)
+			(do_not_autoplace no)
 			(effects
 				(font
@@
 		(property "Sheetfile" "Peripherals.kicad_sch"
 			(at 24.13 55.8296 0)
+			(show_name no)
+			(do_not_autoplace no)
 			(effects
 				(font
@@
 			)
 		)
-		(pin "V4" output
-			(at 55.88 39.37 0)
+		(pin "PSU1" output
+			(at 55.88 31.75 0)
 			(effects
 				(font
@@
 			)
 		)
-		(pin "V2" output
+		(pin "PSU2" output
 			(at 55.88 34.29 0)
 			(effects
@@
 			)
 		)
-		(pin "V3" output
+		(pin "PSU3" output
 			(at 55.88 36.83 0)
 			(effects
@@
 			)
 		)
-		(pin "V1" output
-			(at 55.88 31.75 0)
+		(pin "PSU4" output
+			(at 55.88 39.37 0)
 			(effects
 				(font
@@
 		)
 		(fill
-			(color 0 0 0 0.0000)
+			(color 0 0 0 0)
 		)
 		(property "Sheetname" "Power"
 			(at 67.945 28.4984 0)
+			(show_name no)
+			(do_not_autoplace no)
 			(effects
 				(font
@@
 		(property "Sheetfile" "Power.kicad_sch"
 			(at 67.945 55.8296 0)
+			(show_name no)
+			(do_not_autoplace no)
 			(effects
 				(font
@@
 		)
 		(fill
-			(color 0 0 0 0.0000)
+			(color 0 0 0 0)
 		)
 		(property "Sheetname" "Connector"
 			(at 150.495 29.1334 0)
+			(show_name no)
+			(do_not_autoplace no)
 			(effects
 				(font
@@
 		(property "Sheetfile" "connector.kicad_sch"
 			(at 150.495 55.8296 0)
+			(show_name no)
+			(do_not_autoplace no)
 			(effects
 				(font
@@
 			)
 		)
-		(pin "V1" input
+		(pin "PSU1" input
 			(at 184.15 33.02 0)
 			(effects
@@
 			)
 		)
-		(pin "V2" input
+		(pin "PSU2" input
 			(at 184.15 35.56 0)
 			(effects
@@
 			)
 		)
-		(pin "V3" input
+		(pin "PSU3" input
 			(at 184.15 38.1 0)
 			(effects
@@
 			)
 		)
-		(pin "V4" input
+		(pin "PSU4" input
 			(at 184.15 40.64 0)
 			(effects
@@
 		)
 		(fill
-			(color 0 0 0 0.0000)
+			(color 0 0 0 0)
 		)
 		(property "Sheetname" "MCU"
 			(at 109.22 28.4984 0)
+			(show_name no)
+			(do_not_autoplace no)
 			(effects
 				(font
@@
 		(property "Sheetfile" "MCU.kicad_sch"
 			(at 109.22 56.4646 0)
+			(show_name no)
+			(do_not_autoplace no)
 			(effects
 				(font

Commit message: First review of base module done
Other:
- note added: "Notes: - Make capacitors to common size (100n / 10u --> 1u or 10u) - Check layout of the PAC sensors (in the lib was the wrong package) - Make common symbols for the connectors staff - Where is the resistor-circuit / path to auto-detect the connected FPGA? - Check the questions on the connectors sheet"
Changed lines of the file:
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@@
+		)
+	)
+	(text "Notes:\n- Make capacitors to common size (100n / 10u --> 1u or 10u)\n- Check layout of the PAC sensors (in the lib was the wrong package)\n- Make common symbols for the connectors staff\n- Where is the resistor-circuit / path to auto-detect the connected FPGA?\n- Check the questions on the connectors sheet"
+		(exclude_from_sim no)
+		(at 179.578 163.83 0)
+		(effects
+			(font
+				(size 1.27 1.27)
+			)
+			(justify left bottom)
 		)
 	)
