File: v6/ENV6_DemoBoard_1/Peripherals.kicad_sch (KiCad schematic)
At the start: 34 parts, among them J201 Micro_SD_Card, U201 PAC1954x-x4MX, U202 PAC1954x-x4MX, U203 PAC1954x-x4MX

Commit message: first rev Base Board pcb layout
Parts:
- removed J201: Micro_SD_Card, connectors:microSD_HC_Wuerth_693072010801, symbol connectors:Micro_SD_Card
- added J201: MEM2052-00-195-00-A, ui_stuff:MEM20520019500A, symbol MEM2052-00-195-00-A:MEM2052-00-195-00-A
Connections:
- net GND: now also J201.6 (VSS), J201.9 (SHIELD), J201.G1 (GND_1), J201.G2 (GND_2), J201.G3 (GND_3), J201.G4 (GND_4)
- net GP36/SPI0_RX: now also J201.7 (DAT0)
- net GP37/SPI0_CS: now also J201.2 (CD/DAT3)
- net GP38/SPI0_SCK: now also J201.5 (CLK)
- net GP39/SPI0_TX: now also J201.3 (CMD)
- net PSU_OUT1: now also R210.2, U202.8 (SENSE3+); no longer R208.2, U202.11 (SENSE1+)
- net PSU_OUT2: now also R211.2, U202.10 (SENSE4+); no longer R209.2, U202.13 (SENSE2+)
- net PSU_OUT3: now also R209.2, U202.13 (SENSE2+); no longer R210.2, U202.8 (SENSE3+)
- net PSU_OUT4: now also R208.2, U202.11 (SENSE1+); no longer R211.2, U202.10 (SENSE4+)
- net VDDD_FLASH: now also R202.1, U201.14 (SENSE2-); no longer R203.1, U201.7 (SENSE3-)
- net VDDD_MCU: now also R204.1, U201.9 (SENSE4-); no longer R201.1, U201.12 (SENSE1-)
- net VDDD_PERI: now also R201.1, U201.12 (SENSE1-), J201.4 (VDD); no longer R204.1, U201.9 (SENSE4-)
- net VDDD_RADIO: now also R203.1, U201.7 (SENSE3-); no longer R202.1, U201.14 (SENSE2-)
- net VDIG_IN: now also R216.1, U203.12 (SENSE1-); no longer R217.1, U203.14 (SENSE2-)
- net VFPGA_IN: now also R217.1, U203.14 (SENSE2-); no longer R216.1, U203.12 (SENSE1-)
- net VPERI_IN: now also R215.1, U203.9 (SENSE4-); no longer R218.1, U203.7 (SENSE3-)
- net VSYS_EX: now also R218.1, U203.7 (SENSE3-); no longer R215.1, U203.9 (SENSE4-)
- net V1 renamed PSU4
- net V2 renamed PSU3
- net V3 renamed PSU1
- net V4 renamed PSU2

Commit message: First review of base module done
Parts:
- R201, R202, R203, R204, R208, R209, R210, R211, R215, R216, R217, R218: value 0R82 -> 1R
Other:
- note added: "For shunt resistors: use 0.1%, 1W"
- note removed: "Sensing PAC #3(FPGA board) - FPGA core (1V8) - FPGA core (1V1) - FPGA peripherie (3V3) - FPGA IO-banks + flash (3V3) Acutally it is doubled, maybe remove it?"
- note removed: "find a link to buy sense resistors (0.1% accuracy, high power budget)"
Changed lines of the file:
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@@
 		)
 	)
-	(text "find a link to buy sense resistors \n(0.1% accuracy, high power budget)"
+	(text "For shunt resistors:\nuse 0.1%, 1W"
 		(exclude_from_sim no)
-		(at 32.512 81.534 0)
+		(at 36.83 24.638 0)
 		(effects
 			(font
 				(size 1.27 1.27)
 			)
+			(justify left)
 		)
 	)
@@
 		)
 	)
-	(text "Sensing PAC #3(FPGA board)\n- FPGA core (1V8)\n- FPGA core (1V1)\n- FPGA peripherie (3V3)\n- FPGA IO-banks + flash (3V3)\nAcutally it is doubled, maybe remove it?"
-		(exclude_from_sim no)
-		(at 192.278 105.156 0)
-		(effects
-			(font
-				(size 1.27 1.27)
-			)
-			(justify left top)
-		)
-	)
 	(text "PAC1954 (3)"
 		(exclude_from_sim no)
@@
 	(wire
 		(pts
-			(xy 22.86 115.57) (xy 22.86 116.84)
-		)
-		(stroke
-			(width 0)
-			(type default)
-		)
-	)
-	(wire
-		(pts
 			(xy 34.29 176.53) (xy 35.56 176.53)
 		)
@@
 	(wire
 		(pts
-			(xy 22.86 106.68) (xy 22.86 107.95)
-		)
-		(stroke
-			(width 0)
-			(type default)
-		)
-	)
-	(wire
-		(pts
 			(xy 35.56 60.96) (xy 44.45 60.96)
 		)
@@
 	(wire
 		(pts
-			(xy 22.86 133.35) (xy 22.86 134.62)
-		)
-		(stroke
-			(width 0)
-			(type default)
-		)
-	)
-	(wire
-		(pts
 			(xy 78.74 128.27) (xy 71.12 128.27)
 		)
@@
 	(wire
 		(pts
-			(xy 22.86 124.46) (xy 22.86 125.73)
-		)
-		(stroke
-			(width 0)
-			(type default)
-		)
-	)
-	(wire
-		(pts
 			(xy 114.3 44.45) (xy 114.3 43.18)
 		)
@@
 	(hierarchical_label "PSU1"
 		(shape output)
-		(at 22.86 124.46 180)
+		(at 22.86 125.73 180)
 		(effects
 			(font
@@
 	(hierarchical_label "PSU3"
 		(shape output)
-		(at 22.86 115.57 180)
+		(at 22.86 116.84 180)
 		(effects
 			(font
@@
 	(hierarchical_label "PSU4"
 		(shape output)
-		(at 22.86 106.68 180)
+		(at 22.86 107.95 180)
 		(effects
 			(font
@@
 	(hierarchical_label "PSU2"
 		(shape output)
-		(at 22.86 133.35 180)
+		(at 22.86 134.62 180)
 		(effects
 			(font
@@
 			)
 		)
-		(property "Value" "0R82"
+		(property "Value" "1R"
 			(at 27.94 129.794 90)
 			(show_name no)
@@
 			)
 		)
-		(property "Value" "0R82"
+		(property "Value" "1R"
 			(at 28.956 183.134 90)
 			(show_name no)
@@
 			)
 		)
-		(property "Value" "0R82"
+		(property "Value" "1R"
 			(at 27.94 120.904 90)
 			(show_name no)
@@
 			)
 		)
-		(property "Value" "0R82"
+		(property "Value" "1R"
 			(at 27.94 112.014 90)
 			(show_name no)
@@
 			)
 		)
-		(property "Value" "0R82"
+		(property "Value" "1R"
 			(at 30.48 49.784 90)
 			(show_name no)
@@
 			)
 		)
-		(property "Value" "0R82"
+		(property "Value" "1R"
 			(at 30.48 40.894 90)
 			(show_name no)
@@
 			)
 		)
-		(property "Value" "0R82"
+		(property "Value" "1R"
 			(at 30.48 58.674 90)
 			(show_name no)
@@
 			)
 		)
-		(property "Value" "0R82"
+		(property "Value" "1R"
 			(at 30.48 67.564 90)
 			(show_name no)
@@
 			)
 		)
-		(property "Value" "0R82"
+		(property "Value" "1R"
 			(at 27.94 103.124 90)
 			(show_name no)
@@
 			)
 		)
-		(property "Value" "0R82"
+		(property "Value" "1R"
 			(at 30.226 165.354 90)
 			(show_name no)
@@
 			)
 		)
-		(property "Value" "0R82"
+		(property "Value" "1R"
 			(at 30.226 174.244 90)
 			(show_name no)
@@
 			)
 		)
-		(property "Value" "0R82"
+		(property "Value" "1R"
 			(at 30.226 156.464 90)
 			(show_name no)
