File: v6/ENV6_DemoBoard_1/MCU.kicad_sch (KiCad schematic)
At the start: 41 parts, among them J401 Pico Debugger (SWD), J402 Conn_01x04_Pin, U401 RP2354B, U402 Pi-Radio, U403 W25Q16JVUXIQ, Y401 KX7_QRZ

Commit message: first rev Base Board pcb layout
Parts:
- J401: footprint Connector_PinHeader_2.54mm:PinHeader_1x03_P2.54mm_Vertical -> Connector_PinHeader_2.00mm:PinHeader_1x03_P2.00mm_Vertical
Connections:
- net Unused_GP31 is gone; now on net MCU_LEDS: U401.39 (GPIO_31)
- net MCU_LEDS: no longer U401.27 (GPIO_26)
- net MCU-FPGA_NRST_LOGIC renamed FPGA_RST
- net MCU16-FPGA renamed JTAG_TDI_GP16
- net MCU17-FPGA renamed JTAG_TDO_GP17
- net MCU18-FPGA renamed JTAG_TCK_GP18
- net MCU19-FPGA renamed JTAG_TMS_GP19
- net V_SYS renamed VPERI_IN
- new net Unused_GP26: U401.27 (GPIO_26)
- no-connect marks 3 -> 4

Commit message: First review of base module done
Other:
- note removed: "Infos for FPGA board - Adding Testpads to all these signals on the FPGA board - Add ADC for identifying which FPGA board is connected via voltage divider - Move F_Mx pins to fpga directly (configure flash fpga interaction) using resistors - One Clock Oscillator with enable pin - One RSTN button for the FPGA logic - Bring unused GPIO to connector (for application)"
Changed lines of the file:
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@@
 		)
 	)
-	(text "Infos for FPGA board\n- Adding Testpads to all these signals on the FPGA board\n- Add ADC for identifying which FPGA board is connected via voltage divider\n- Move F_Mx pins to fpga directly (configure flash fpga interaction) using resistors\n- One Clock Oscillator with enable pin\n- One RSTN button for the FPGA logic\n- Bring unused GPIO to connector (for application)"
-		(exclude_from_sim no)
-		(at 105.664 186.944 0)
-		(effects
-			(font
-				(size 1.27 1.27)
-			)
-			(justify left top)
-		)
-	)
 	(text "DirtyJTAG\nFor FPGA"
 		(exclude_from_sim no)
@@
 		(fields_autoplaced yes)
 		(property "Reference" "S401"
-			(at 187.96 49.53 0)
+			(at 196.85 48.26 90)
 			(show_name no)
 			(do_not_autoplace no)
@@
 					(size 1.778 1.5113)
 				)
+				(justify right)
 			)
 		)
 		(property "Value" "MCU_RSTN"
-			(at 190.5 49.53 0)
+			(at 196.85 51.4349 90)
 			(show_name no)
 			(do_not_autoplace no)
@@
 					(size 1.27 1.27)
 				)
+				(justify right)
 			)
 		)
@@
 		(fields_autoplaced yes)
 		(property "Reference" "S402"
-			(at 245.11 49.53 0)
+			(at 254 48.26 90)
 			(show_name no)
 			(do_not_autoplace no)
@@
 					(size 1.778 1.5113)
 				)
+				(justify right)
 			)
 		)
 		(property "Value" "BTN"
-			(at 247.65 49.53 0)
+			(at 254 51.4349 90)
 			(show_name no)
 			(do_not_autoplace no)
@@
 					(size 1.27 1.27)
 				)
+				(justify right)
 			)
 		)

Commit message: updated Baseboard
Parts:
- added NT401: NetTie_2, NetTie:NetTie-2_SMD_Pad0.5mm, symbol Device:NetTie_2
Connections:
- net GND: now also NT401.1; no longer C417.1, C418.1, Y401.2 (SH), Y401.4 (SH)
- new net OSCGND: C417.1, C418.1, NT401.2, Y401.2 (SH), Y401.4 (SH)
Changed lines of the file:
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@@
 			)
 		)
-		(property "Value" "GND"
+		(property "Value" "OSCGND"
 			(at 85.09 185.42 0)
 			(show_name no)
@@
 				(path "/c353698e-fca1-4ed3-95bc-4f5142868012/ed3a85d8-235b-4bef-8433-9f631d48a830"
 					(reference "Y401")
+					(unit 1)
+				)
+			)
+		)
+	)
+	(symbol
+		(lib_id "power:GND")
+		(at 73.66 193.04 270)
+		(unit 1)
+		(body_style 1)
+		(exclude_from_sim no)
+		(in_bom yes)
+		(on_board yes)
+		(in_pos_files yes)
+		(dnp no)
+		(property "Reference" "#PWR0418"
+			(at 67.31 193.04 0)
+			(hide yes)
+			(show_name no)
+			(do_not_autoplace no)
+			(effects
+				(font
+					(size 1.27 1.27)
+				)
+			)
+		)
+		(property "Value" "GND"
+			(at 68.834 193.04 90)
+			(show_name no)
+			(do_not_autoplace no)
+			(effects
+				(font
+					(size 1.27 1.27)
+				)
+			)
+		)
+		(property "Footprint" ""
+			(at 73.66 193.04 0)
+			(hide yes)
+			(show_name no)
+			(do_not_autoplace no)
+			(effects
+				(font
+					(size 1.27 1.27)
+				)
+			)
+		)
+		(property "Datasheet" ""
+			(at 73.66 193.04 0)
+			(hide yes)
+			(show_name no)
+			(do_not_autoplace no)
+			(effects
+				(font
+					(size 1.27 1.27)
+				)
+			)
+		)
+		(property "Description" "Power symbol creates a global label with name \"GND\" , ground"
+			(at 73.66 193.04 0)
+			(hide yes)
+			(show_name no)
+			(do_not_autoplace no)
+			(effects
+				(font
+					(size 1.27 1.27)
+				)
+			)
+		)
+		(pin "1"
+		)
+		(instances
+			(project "ENV6_DemoBoard_1"
+				(path "/c353698e-fca1-4ed3-95bc-4f5142868012/ed3a85d8-235b-4bef-8433-9f631d48a830"
+					(reference "#PWR0418")
 					(unit 1)
 				)
@@
 	)
 	(symbol
+		(lib_id "Device:NetTie_2")
+		(at 76.2 193.04 0)
+		(unit 1)
+		(body_style 1)
+		(exclude_from_sim no)
+		(in_bom no)
+		(on_board yes)
+		(in_pos_files yes)
+		(dnp no)
+		(fields_autoplaced yes)
+		(property "Reference" "NT401"
+			(at 76.2 187.96 0)
+			(show_name no)
+			(do_not_autoplace no)
+			(effects
+				(font
+					(size 1.27 1.27)
+				)
+			)
+		)
+		(property "Value" "NetTie_2"
+			(at 76.2 190.5 0)
+			(show_name no)
+			(do_not_autoplace no)
+			(effects
+				(font
+					(size 1.27 1.27)
+				)
+			)
+		)
+		(property "Footprint" "NetTie:NetTie-2_SMD_Pad0.5mm"
+			(at 76.2 193.04 0)
+			(hide yes)
+			(show_name no)
+			(do_not_autoplace no)
+			(effects
+				(font
+					(size 1.27 1.27)
+				)
+			)
+		)
+		(property "Datasheet" ""
+			(at 76.2 193.04 0)
+			(hide yes)
+			(show_name no)
+			(do_not_autoplace no)
+			(effects
+				(font
+					(size 1.27 1.27)
+				)
+			)
+		)
+		(property "Description" "Net tie, 2 pins"
+			(at 76.2 193.04 0)
+			(hide yes)
+			(show_name no)
+			(do_not_autoplace no)
+			(effects
+				(font
+					(size 1.27 1.27)
+				)
+			)
+		)
+		(pin "2"
+		)
+		(pin "1"
+		)
+		(instances
+			(project "ENV6_DemoBoard_1"
+				(path "/c353698e-fca1-4ed3-95bc-4f5142868012/ed3a85d8-235b-4bef-8433-9f631d48a830"
+					(reference "NT401")
+					(unit 1)
+				)
+			)
+		)
+	)
+	(symbol
 		(lib_id "passive:C0402")
 		(at 43.18 58.42 180)
@@
 					(unit 1)
 				)
+			)
+		)
+	)
+	(symbol
+		(lib_id "power:GND")
+		(at 78.74 193.04 90)
+		(unit 1)
+		(body_style 1)
+		(exclude_from_sim no)
+		(in_bom yes)
+		(on_board yes)
+		(in_pos_files yes)
+		(dnp no)
+		(property "Reference" "#PWR0419"
+			(at 85.09 193.04 0)
+			(hide yes)
+			(show_name no)
+			(do_not_autoplace no)
+			(effects
+				(font
+					(size 1.27 1.27)
+				)
+			)
+		)
+		(property "Value" "OSCGND"
+			(at 85.598 193.04 90)
+			(show_name no)
+			(do_not_autoplace no)
+			(effects
+				(font
+					(size 1.27 1.27)
+				)
+			)
+		)
+		(property "Footprint" ""
+			(at 78.74 193.04 0)
+			(hide yes)
+			(show_name no)
+			(do_not_autoplace no)
+			(effects
+				(font
+					(size 1.27 1.27)
+				)
+			)
+		)
+		(property "Datasheet" ""
+			(at 78.74 193.04 0)
+			(hide yes)
+			(show_name no)
+			(do_not_autoplace no)
+			(effects
+				(font
+					(size 1.27 1.27)
+				)
+			)
+		)
+		(property "Description" "Power symbol creates a global label with name \"GND\" , ground"
+			(at 78.74 193.04 0)
+			(hide yes)
+			(show_name no)
+			(do_not_autoplace no)
+			(effects
+				(font
+					(size 1.27 1.27)
+				)
+			)
+		)
+		(pin "1"
+		)
+		(instances
+			(project "ENV6_DemoBoard_1"
+				(path "/c353698e-fca1-4ed3-95bc-4f5142868012/ed3a85d8-235b-4bef-8433-9f631d48a830"
+					(reference "#PWR0419")
+					(unit 1)
+				)
