File: v6/ENV6_DemoBoard_1/connector.kicad_sch (KiCad schematic)
At the start: 9 parts, among them J501 Conn_02x16_Odd_Even, J502 Conn_02x04_Odd_Even, J503 Conn_02x16_Odd_Even, J504 Conn_02x04_Odd_Even, J505 Conn_02x16_Odd_Even

Commit message: first rev Base Board pcb layout
Connections:
- net Unused_GP31 is gone; now on net VDDD_MCU: J501.30 (Pin_30)
- net GND: now also J505.20 (Pin_20), J505.31 (Pin_31), J505.32 (Pin_32); no longer J505.21 (Pin_21)
- net VDDD_MCU: now also J505.21 (Pin_21); no longer J501.29 (Pin_29)
- net VDDD_PERI: no longer J505.20 (Pin_20)
- net V1 renamed PSU1
- net V2 renamed PSU2
- net V3 renamed PSU4
- net V4 renamed PSU3
- net V_App_Board: no longer names the net of J505.23 (Pin_23)
- net V_App_Board: no longer J505.24 (Pin_24)
- new net Unused_GP26: J501.29 (Pin_29)

Commit message: First review of base module done
Other:
- note added: "Questions: - Which function has FPGA_RST? Logic RST or Config-RST? - Where can I readout which FPGA is connected? - Clock is placed on the other board, right? --> Maybe make a list / sheet with the function of each pin"
- note removed: "Add these pins to the FPGA board"
Changed lines of the file:
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@@
+		)
+	)
+	(text "Questions:\n- Which function has FPGA_RST? Logic RST or Config-RST?\n- Where can I readout which FPGA is connected?\n- Clock is placed on the other board, right?\n--> Maybe make a list / sheet with the function of each pin"
+		(exclude_from_sim no)
+		(at 124.46 17.272 0)
+		(effects
+			(font
+				(size 1.27 1.27)
+			)
 		)
 	)
@@
 		(effects
 			(font
-				(size 1.27 1.27)
-			)
-		)
-	)
-	(text "Add these pins to the FPGA board"
-		(exclude_from_sim no)
-		(at 75.184 195.834 0)
-		(effects
-			(font

Commit message: updated Baseboard
Changed lines of the file:
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@@
 	(text "Questions:\n- Which function has FPGA_RST? Logic RST or Config-RST?\n- Where can I readout which FPGA is connected?\n- Clock is placed on the other board, right?\n--> Maybe make a list / sheet with the function of each pin"
 		(exclude_from_sim no)
-		(at 124.46 17.272 0)
+		(at 118.618 13.97 0)
 		(effects
 			(font
